File: BusinessCard.kicad_pcb (KiCad board)
At the start: 2 copper layers, 74 x 74 mm, 19 parts, among them U2 ST25DV64K-IER8C3

Commit message: added docs
Parts:
- AE1: value Antenna_Loop -> NFC Antenna
- D1: value LED -> Red
- U2: value ST25DV64K-IER8C3 -> ST25DV04K
