File: BusinessCard.kicad_sch (KiCad schematic)
At the start: 15 parts, among them U2 ST25DV64K-IER8C3

Commit message: added docs
Parts:
- AE1: value Antenna_Loop -> NFC Antenna
- U2: value ST25DV64K-IER8C3 -> ST25DV04K
Changed lines of the file:
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@@
 			)
 		)
-		(property "Value" "Antenna_Loop"
+		(property "Value" "NFC Antenna"
 			(at 151.13 68.5801 90)
 			(effects
@@
 			)
 		)
-		(property "Value" "ST25DV64K-IER8C3"
+		(property "Value" "ST25DV04K"
 			(at 108.204 78.232 0)
 			(effects
